Commit message: Added virtual end point to the arm

File: ros_workspace/src/popsicle_arm/urdf/popsicle_bot.urdf (robot description, URDF)
Before this commit: robot popsicle_bot, 8 links, 7 joints
Links:
- added link end; visual box size=0.0135 0.0135 0.0135
Joints:
- added joint m2_arm_to_end: type fixed, parent m2_arm, child end, origin xyz=0 0 0.115

File: ros_workspace/src/popsicle_arm/urdf/popsicle_bot.xacro (robot description, xacro)
@@ -152,3 +152,19 @@
         </visual>
     </link>
+    <joint name="m2_arm_to_end" type="fixed">
+        <parent link="m2_arm"/>
+        <child link="end"/>
+        <origin xyz="0 0 ${stick_length}"/>
+    </joint>
+    <link name="end">
+        <visual>
+            <geometry>
+                <box size="${stick_width*1.5} ${stick_width*1.5} ${stick_width*1.5}"/>
+            </geometry>
+            <origin xyz="0 0 0"/>
+            <material name="end">
+                <color rgba="0.0 0.0 1.0 0.5"/>
+            </material>
+        </visual>
+    </link>
 </robot>

Commit message: Added files as a quick backup. JointTarget message can be used to move arm to a location

File: ros_workspace/src/popsicle_arm/urdf/popsicle_bot.urdf (robot description, URDF)
Before this commit: robot popsicle_bot, 9 links, 8 joints
Links:
- added link virtual_main_stop; collision box size=0.002 0.009 0.11; visual box size=0.009 0.009 0.11
- link base_link: geometry collision box size=0.2 0.28 0.06; visual box size=0.2 0.28 0.06
- link m1_arm: geometry collision box size=0.002 0.009 0.115; visual box size=0.002 0.009 0.115
- link m2_arm: geometry collision box size=0.002 0.009 0.115; visual box size=0.002 0.009 0.115
- link main_stand: geometry collision box size=0.002 0.009 0.11; visual box size=0.002 0.009 0.11
- link plastic_1: geometry collision box size=0.0027 0.038 0.023; visual box size=0.0027 0.038 0.023
- link plastic_2: geometry collision box size=0.0027 0.038 0.023; visual box size=0.0027 0.038 0.023
Joints:
- added joint main_stand_to_virtual_main_stop: type fixed, parent main_stand, child virtual_main_stop, origin xyz=0 0.018 0
- joint m2_arm_to_end: type fixed -> continuous

File: ros_workspace/src/popsicle_arm/urdf/popsicle_bot.xacro (robot description, xacro)
@@ -40,4 +40,9 @@
         </material>
     </xacro:macro>
+    <xacro:macro name="material_virtual">
+        <material name="virtual_stop">
+            <color rgba="0.5 0.5 0.0 0.5"/>
+        </material>
+    </xacro:macro>
     <link name="base_link">
         <visual>
@@ -46,6 +51,12 @@
             </geometry>
             <origin xyz="${base_size_x/2.0} ${-base_size_y/2.0} ${base_size_z/2.0}"/>
-        <xacro:material_black/>
-        </visual>
+            <xacro:material_black/>
+        </visual>
+        <collision>
+            <geometry>
+                <box size="${base_size_x} ${base_size_y} ${base_size_z}"/>
+            </geometry>
+            <origin xyz="${base_size_x/2.0} ${-base_size_y/2.0} ${base_size_z/2.0}"/>
+        </collision>
     </link>
     <joint name="base_to_main_stand" type="fixed">
@@ -60,7 +71,33 @@
             </geometry>
             <origin xyz="0 0 ${main_stand_height/2.0}"/>
-        <xacro:material_popsicle/>
-        </visual>
-    </link>
+            <xacro:material_popsicle/>
+        </visual>
+        <collision>
+            <geometry>
+                <box size="${stick_width_small} ${stick_width} ${main_stand_height}"/>
+            </geometry>
+            <origin xyz="0 0 ${main_stand_height/2.0}"/>
+        </collision>
+    </link>
+    <link name="virtual_main_stop">
+        <visual>
+            <geometry>
+                <box size="${stick_width} ${stick_width} ${main_stand_height}"/>
+            </geometry>
+            <origin xyz="${stick_width} ${stick_width} ${main_stand_height/2.0}"/>
+            <xacro:material_virtual/>
+        </visual>
+        <collision>
+            <geometry>
+                <box size="${stick_width_small} ${stick_width} ${main_stand_height}"/>
+            </geometry>
+            <origin xyz="0 0 ${main_stand_height/2.0}"/>
+        </collision>
+    </link>
+    <joint name="main_stand_to_virtual_main_stop" type="fixed">
+        <parent link="main_stand"/>
+        <child link="virtual_main_stop"/>
+        <origin xyz="0 ${stick_width*2} 0"/>
+    </joint>
     <joint name="main_stand_to_motor_1" type="fixed">
         <parent link="main_stand"/>
@@ -92,6 +129,12 @@
             </geometry>
             <origin xyz="0.0 ${-plastic_y/2.0+0.01} 0"/>
-        <xacro:material_black/>
-        </visual>
+            <xacro:material_black/>
+        </visual>
+        <collision>
+            <geometry>
+                <box size="${plastic_x} ${plastic_y} ${plastic_z}"/>
+            </geometry>
+            <origin xyz="0.0 ${-plastic_y/2.0+0.01} 0"/>
+        </collision>
     </link>
     <joint name="plastic_1_to_m1_arm" type="fixed">
@@ -108,4 +151,10 @@
             <xacro:material_popsicle/>
         </visual>
+        <collision>
+            <geometry>
+                <box size="${stick_width_small} ${stick_width} ${stick_length}"/>
+            </geometry>
+            <origin xyz="0 0 ${stick_length/2.0}"/>
+        </collision>
     </link>
     <joint name="m1_arm_to_motor_2" type="fixed">
@@ -135,6 +184,12 @@
             </geometry>
             <origin xyz="0.0 ${-plastic_y/2.0+0.01} 0"/>
-        <xacro:material_black/>
-        </visual>
+            <xacro:material_black/>
+        </visual>
+        <collision>
+            <geometry>
+                <box size="${plastic_x} ${plastic_y} ${plastic_z}"/>
+            </geometry>
+            <origin xyz="0.0 ${-plastic_y/2.0+0.01} 0"/>
+        </collision>
     </link>
     <joint name="plastic_2_to_m2_arm" type="fixed">
@@ -151,6 +206,12 @@
             <xacro:material_popsicle/>
         </visual>
-    </link>
-    <joint name="m2_arm_to_end" type="fixed">
+        <collision>
+            <geometry>
+                <box size="${stick_width_small} ${stick_width} ${stick_length}"/>
+            </geometry>
+            <origin xyz="0 0 ${stick_length/2.0}"/>
+        </collision>
+    </link>
+    <joint name="m2_arm_to_end" type="continuous">
         <parent link="m2_arm"/>
         <child link="end"/>
